Commit message: backup

File: orne_description/urdf/alpha/orne_alpha.urdf.xacro (robot description, xacro)
@@ -32,5 +32,5 @@
     </visual>
     <collision>
-      <origin xyz="0.005 0 0.300" rpy="0 0 0"/>
+      <origin xyz="0.005 0 0.305" rpy="0 0 0"/>
       <geometry>
 	       <box size=".376 .40 .134"/>
@@ -80,23 +80,8 @@
   <!-- Setting for levelly fixed 2D URG -->
   <xacro:sensor_hokuyo name="hokuyo" parent="base_link" size="0.05 0.05 0.05">
-      <origin xyz="0.212 0 0.375" rpy="0 0 0"/>
+      <origin xyz="0.212 0 0.2485" rpy="0 0 0"/>
   </xacro:sensor_hokuyo>
-  <!-- <link name="visual_left_wheel">
-    <visual name="visual">
-      <origin xyz="0 0.0 0" rpy="0 1.5707 1.5707"/>
-      <geometry>
-        <cylinder  length="0.03" radius="0.151"/>
-      </geometry>
-    </visual>
-  </link> -->
-  <!-- <joint type="fixed" name="visual_left_wheel_joint">
-    <origin xyz="-0.045 0.233 0.1518" rpy="0 0 0"/>
-    <child link="visual_left_wheel">visual_left_wheel</child>
-    <parent link="base_link">base_link</parent>
-    <axis xyz="0 1 0"/>
-  </joint> -->
   <link name="left_wheel">
     <collision name="collision">
-      <!-- <origin xyz="0 0.0 0" rpy="0 1.5707 1.5707"/> -->
       <origin xyz="0 0.0 0" rpy="0 0 0"/>
       <geometry>
@@ -105,5 +90,4 @@
     </collision>
     <visual name="visual">
-      <!-- <origin xyz="0 0.0 0" rpy="0 1.5707 1.5707"/> -->
       <origin xyz="0 0.0 0" rpy="0 0 0"/>
       <geometry>
@@ -124,18 +108,4 @@
     <limit effort="100" velocity="100.0"  lower="-5000" upper="5000" />
   </joint>
-  <!-- <link name="visual_right_wheel">
-    <visual name="visual">
-      <origin xyz="0 0.0 0" rpy="0 1.5707 1.5707"/>
-      <geometry>
-        <cylinder  length="0.03" radius="0.151"/>
-      </geometry>
-    </visual>
-  </link> -->
-  <!-- <joint type="fixed" name="visual_right_wheel_joint">
-    <origin xyz="-0.045 -0.223 0.1518" rpy="0 0 0"/>
-    <child link="visual_right_wheel">visual_right_wheel</child>
-    <parent link="base_link">base_link</parent>
-    <axis xyz="0 1 0"/>
-  </joint> -->
   <link name="right_wheel">
     <collision name="collision">

File: orne_description/urdf/sensors/imu.urdf.xacro (robot description, xacro)
@@ -22,7 +22,7 @@
       </visual>
     </link>
-      <!-- <gazebo>
+      <gazebo>
         <plugin name="ros_imu" filename="libgazebo_ros_imu.so">
-          <bodyName>${parent}</bodyName>
+          <bodyName>${parent}</bodyName> <!-- bodyName always set base_link by URDF parser -->
           <topicName>imu_data</topicName>
           <serviceName>imu_service</serviceName>
@@ -32,5 +32,4 @@
         </plugin>
       </gazebo>
-    -->
   </xacro:macro>
 </robot>
