Commit message: refactor gamma and navifgation

File: orne_description/urdf/gamma/orne_gamma.urdf.xacro (robot description, xacro)
@@ -20,5 +20,5 @@
     <visual>
       <!-- <origin xyz="-0.15 0 0.1" rpy="0 0 0"/> -->
-      <origin xyz="0.0 0.0 0.0" rpy="0.0 0.0 0.0"/>>
+      <origin xyz="0.0 0.0 0.0" rpy="0.0 0.0 0.0"/>
       <geometry>
 	    <box size=".485 .43 .15"/>
@@ -28,5 +28,5 @@
     <collision name="collision">
       <!-- <origin xyz="-0.15 0 0.1" rpy="0 0 0"/> -->
-      <origin xyz="0.0 0.0 0.0" rpy="0.0 0.0 0.0"/>>
+      <origin xyz="0.0 0.0 0.0" rpy="0.0 0.0 0.0"/>
       <geometry>
 	    <box size=".485 .43 .15"/>

Commit message: backup

File: orne_description/urdf/gamma/orne_gamma.urdf.xacro (robot description, xacro)
@@ -203,5 +203,6 @@
   </transmission>
   <joint name="camera_joint" type="fixed">
-    <origin xyz="0.223 -0.011 0.565" rpy="0 0.124 0"/>
+    <!-- <origin xyz="0.223 -0.011 0.565" rpy="0 0.124 0"/>  -->
+    <origin xyz="0.223 -0.011 0.394" rpy="0 0.124 0"/>
     <parent link="base_link"/>
     <child link="camera_link"/>

Commit message: add real_environment

File: orne_description/urdf/gamma/orne_gamma.urdf.xacro (robot description, xacro)
@@ -1,5 +1,5 @@
 <?xml version="1.0"?>
 <!-- Revolute-Revolute Manipulator -->
-<robot name="orne_gamma" xmlns:xacro="http://ros.org/wiki/xacro">
+<robot name="orne_gamma" xmlns:xacro="http://www.ros.org/wiki/xacro">
   <!-- Constants for robot dimensions -->
   <xacro:property name="PI" value="3.1415926535897931"/>
@@ -8,5 +8,4 @@
   <xacro:include filename="$(find orne_description)/urdf/gamma/orne_gamma.gazebo"/>
   <xacro:include filename="$(find orne_description)/urdf/sensors/hokuyo.urdf.xacro"/>
-  <xacro:include filename="$(find orne_description)/urdf/gamma/orne_gamma_caster.urdf.xacro"/>
   <!--Base Footprint-->
   <link name="base_footprint" />
@@ -20,5 +19,5 @@
     <visual>
       <!-- <origin xyz="-0.15 0 0.1" rpy="0 0 0"/> -->
-      <origin xyz="0.0 0.0 0.0" rpy="0.0 0.0 0.0"/>
+      <origin xyz="0.0 0.0 0.0" rpy="0.0 0.0 0.0"/>>
       <geometry>
 	    <box size=".485 .43 .15"/>
@@ -28,10 +27,10 @@
     <collision name="collision">
       <!-- <origin xyz="-0.15 0 0.1" rpy="0 0 0"/> -->
-      <origin xyz="0.0 0.0 0.0" rpy="0.0 0.0 0.0"/>
+      <origin xyz="0.0 0.0 0.0" rpy="0.0 0.0 0.0"/>>
       <geometry>
 	    <box size=".485 .43 .15"/>
       </geometry>
     </collision>
-     <!-- <collision name="collision">
+     <collision name="collision">
       <origin xyz="0.15 0.0 -0.075" rpy="1.57 0.0 0.0"/>
       <geometry>
@@ -44,5 +43,5 @@
         <cylinder  length="0.03" radius="0.04625"/>
       </geometry>
-    </visual> -->
+    </visual>
     <!-- <inertial>
       <mass value="20" />
@@ -53,6 +52,5 @@
     <mass value="15" />
     <origin xyz="0 0 0" rpy="0 0 0"/>
-    <!-- <inertia ixx="0.5" ixy="0" ixz="0" iyy="0.5" iyz="0" izz="0.5" /> -->
-    <inertia ixx="0.25925" ixy="0" ixz="0" iyy="0.32216" iyz="0" izz="0.52516" />
+    <inertia ixx="1" ixy="0" ixz="0" iyy="1" iyz="0" izz="1" />
     </inertial>
  </link>
@@ -97,6 +95,4 @@
     <collision name="collision">
       <!-- <origin xyz="0 0.0 -0.10" rpy="0 1.5707 1.5707"/> -->
-      <!-- <origin xyz="-0.15 0.15 -0.05" rpy="-1.57 0.0 0.0"/> -->
-      <origin xyz="0.0 0.0 0.0" rpy="0.0 0.0 0.0"/>
       <geometry>
          <cylinder  length="0.03" radius="0.0725"/>
@@ -105,6 +101,4 @@
     <visual name="visual">
       <!-- <origin xyz="0 0.0 -0.10" rpy="0 0 0"/> -->
-      <!-- <origin xyz="-0.15 0.15 -0.05" rpy="-1.57 0.0 0.0"/> -->
-      <origin xyz="0.0 0.0 0.0" rpy="0.0 0.0 0.0"/>
       <geometry>
         <cylinder  length="0.03" radius="0.0725"/>
@@ -113,7 +107,6 @@
     <inertial>
       <mass value="1" />
-      <!-- <origin xyz="-0.15 0.15 -0.05" rpy="-1.57 0.0 0.0"/> -->
-      <origin xyz="0.0 0.0 0.0" rpy="0.0 0.0 0.0"/>
-      <inertia ixx="0.001" ixy="0" ixz="0" iyy="0.002" iyz="0" izz="0.001" />
+      <origin xyz="-0.15 0.15 -0.05" rpy="-1.57 0.0 0.0"/>
+      <inertia ixx="0.1" ixy="0" ixz="0" iyy="0.1" iyz="0" izz="0.1" />
     </inertial>
   </link>
@@ -125,5 +118,4 @@
     <axis xyz="0 0 1"/>
     <limit effort="100" velocity="100.0"  lower="-5000" upper="5000" />
-    <dynamics damping="0.1"/>
   </joint>
   <!--link name="visual_right_wheel">
@@ -143,6 +135,4 @@
   <link name="right_wheel">
     <collision name="collision">
-      <!-- <origin xyz="-0.15 -0.15 -0.05" rpy="-1.57 0.0 0.0"/> -->
-      <origin xyz="0.0 0.0 0.0" rpy="0.0 0.0 0.0"/>
       <!-- <origin xyz="0 0.0 -0.10" rpy="0 1.5707 1.5707"/> -->
       <!-- <origin xyz="0 0.15 -0.05" rpy="1.57 0 0"/> -->
@@ -153,6 +143,4 @@
     <visual name="visual">
       <!-- <origin xyz="0 0.0 -0.10" rpy="0 1.5707 1.5707"/> -->
-      <!-- <origin xyz="-0.15 -0.15 -0.05" rpy="-1.57 0.0 0.0"/> -->
-      <origin xyz="0.0 0.0 0.0" rpy="0.0 0.0 0.0"/>
       <geometry>
         <cylinder  length="0.03" radius="0.0725"/>
@@ -161,7 +149,6 @@
     <inertial>
       <mass value="1" />
-      <!-- <origin xyz="-0.15 -0.15 -0.05" rpy="-1.57 0.0 0.0"/> -->
-      <origin xyz="0.0 0.0 0.0" rpy="0.0 0.0 0.0"/>
-      <inertia ixx="0.001" ixy="0" ixz="0" iyy="0.002" iyz="0" izz="0.001" />
+       <origin xyz="-0.15 0.15 -0.05" rpy="-1.57 0.0 0.0"/>
+      <inertia ixx="0.1" ixy="0" ixz="0" iyy="0.1" iyz="0" izz="0.1" />
     </inertial>
   </link>
@@ -174,12 +161,8 @@
     <axis xyz="0 0 1"/>
     <limit effort="100" velocity="100.0"  lower="-5000" upper="5000" />
-    <dynamics damping="0.1"/>
   </joint>
   <xacro:sensor_hokuyo name="hokuyo" parent="base_link" size="0.05 0.05 0.05">
     <origin xyz="0.25 0 0.1" rpy="0 0 0"/>
   </xacro:sensor_hokuyo>
-  <xacro:caster sub="0" parent="base_link" transX="0.15" transY="0.0" transZ="-0.075" />
-    <!-- <origin xyz="0.25 0 0.1" rpy="0 0 0"/> -->
-  <!-- </xacro:caster> -->
   <transmission name="tran1">
     <type>transmission_interface/SimpleTransmission</type>
@@ -202,52 +185,3 @@
     </actuator>
   </transmission>
-  <joint name="camera_joint" type="fixed">
-    <origin xyz="0.223 -0.011 0.565" rpy="0 0.124 0"/>
-    <parent link="base_link"/>
-    <child link="camera_link"/>
-  </joint>
-  <link name="camera_link">
-    <collision>
-      <origin xyz="0.005 0.011 0.013" rpy="0 0 0"/>
-      <geometry>
-        <box size="0.015 0.030 0.027"/>
-      </geometry>
-    </collision>
-  </link>
-  <joint name="camera_rgb_joint" type="fixed">
-    <origin xyz="0.003 0.011 0.009" rpy="0 0 0"/>
-    <parent link="camera_link"/>
-    <child link="camera_rgb_frame"/>
-  </joint>
-  <link name="camera_rgb_frame"/>
-  <joint name="camera_rgb_optical_joint" type="fixed">
-    <origin xyz="0 0 0" rpy="-1.57 0 -1.57"/>
-    <parent link="camera_rgb_frame"/>
-    <child link="camera_rgb_optical_frame"/>
-  </joint>
-  <link name="camera_rgb_optical_frame"/>
-  <joint name="camera_rgb_left_joint" type="fixed">
-    <origin xyz="0.003 0.111 0.009" rpy="0 0 0.175"/>
-    <parent link="camera_link"/>
-    <child link="camera_rgb_left_frame"/>
-  </joint>
-  <link name="camera_rgb_left_frame"/>
-  <joint name="camera_rgb_optical_left_joint" type="fixed">
-    <origin xyz="0 0 0" rpy="-1.57 0 -1.57"/>
-    <parent link="camera_rgb_left_frame"/>
-    <child link="camera_rgb_optical_left_frame"/>
-  </joint>
-  <link name="camera_rgb_optical_left_frame"/>
-  <joint name="camera_rgb_right_joint" type="fixed">
-    <origin xyz="0.003 -0.089 0.009" rpy="0 0 -0.175"/>
-    <parent link="camera_link"/>
-    <child link="camera_rgb_right_frame"/>
-  </joint>
-  <link name="camera_rgb_right_frame"/>
-  <joint name="camera_rgb_optical_right_joint" type="fixed">
-    <origin xyz="0 0 0" rpy="-1.57 0 -1.57"/>
-    <parent link="camera_rgb_right_frame"/>
-    <child link="camera_rgb_optical_right_frame"/>
-  </joint>
-  <link name="camera_rgb_optical_right_frame"/>
 </robot>

File: orne_description/urdf/gamma/orne_gamma_caster.urdf.xacro (robot description, xacro)
@@ -1,43 +1,169 @@
 <?xml version="1.0"?>
-<robot name="caster" xmlns:xacro="http://www.ros.org/wiki/xacro">
-  <!-- Casters -->
-  <xacro:property name="caster_radius" value="0.05250" /> <!-- in m -->
-  <xacro:property name="caster_mass"   value="1.00" /> <!-- in kg-->
-  <xacro:macro name="caster" params="sub parent transX transY transZ">
-    <!-- sub: l,r 0,1,2,3 etc -->
-    <!-- parent: parent link name -->
-    <!-- transX transY transZ: xyz position -->
-    <link name="caster_${sub}">
-      <visual>
-        <origin xyz="0 0 0" rpy="0 0 0" />
-        <geometry>
-          <sphere radius="${caster_radius}" />
-        </geometry>
-        <material name="Black" />
-      </visual>
-      <collision>
-        <origin xyz="0 0 0" rpy="0 0 0" />
-        <geometry>
-          <sphere radius="${caster_radius}" />
-        </geometry>
-      </collision>
-      <inertial>
-        <mass value="${caster_mass}" />
-        <origin xyz="0 0 0" />
-        <!-- <xacro:sphere_inertia m="${caster_mass}" r="${caster_radius}" /> -->
-        <inertia ixx="0.001" ixy="0.0" ixz="0.0" iyy="0.001" iyz="0.0" izz="0.001"/>
-      </inertial>
+<!-- Revolute-Revolute Manipulator -->
+<robot name="orne_gamma" xmlns:xacro="http://www.ros.org/wiki/xacro">
+  <!-- Constants for robot dimensions -->
+  <xacro:property name="PI" value="3.1415926535897931"/>
+  <!-- Import Rviz colors -->
+  <xacro:include filename="$(find orne_box_description)/urdf/material_colors.xacro"/>
+  <xacro:include filename="$(find orne_box_description)/urdf/sensors/hokuyo.urdf.xacro"/>
+  <!--Base Footprint-->
+  <link name="base_footprint" />
+  <joint name="base_joint" type="fixed">
+    <origin xyz="0 0 0" />
+    <parent link="base_footprint" />
+    <child link="base_link" />
+  </joint>
+  <!-- Base Link -->
+  <link name="base_link">
+    <visual>
+      <!-- <origin xyz="-0.15 0 0.1" rpy="0 0 0"/> -->
+      <origin xyz="0.0 0.0 0.0" rpy="0.0 0.0 0.0"/>>
+      <geometry>
+	    <box size=".485 .43 .15"/>
+      </geometry>
+      <!-- <material name="orange"/> -->
+    </visual>
+    <collision>
+      <!-- <origin xyz="-0.15 0 0.1" rpy="0 0 0"/> -->
+      <origin xyz="0.0 0.0 0.0" rpy="0.0 0.0 0.0"/>>
+      <geometry>
+	    <box size=".485 .43 .15"/>
+      </geometry>
+    </collision>
+    <inertial>
+      <mass value="20" />
+      <origin xyz="-0.08 0 0" rpy="0 0 0"/>
+      <inertia ixx="1" ixy="0" ixz="0" iyy="1" iyz="0" izz="1" />
+   </inertial>
+ </link>
+   <link name="caster">
+    <collision name="collision">
+      <!-- <origin xyz="-0.325 0.0 0.05" rpy="0 1.5707 1.5707"/> -->
+      <geometry>
+        <cylinder  length="0.03" radius="0.04625"/>
+      </geometry>
+    </collision>
+    <visual name="visual">
+      <!-- <origin xyz="-0.325 0.0 -0.075" rpy="0 1.5707 1.5707"/> -->
+      <geometry>
+        <cylinder  length="0.03" radius="0.04625"/>
+      </geometry>
+    </visual>
     </link>
-    <gazebo reference="caster_${sub}">
-      <turnGravityOff>false</turnGravityOff>
-      <material>Gazebo/Black</material>
-      <mu1 value="0.0"/>
-      <mu2 value="0.0"/>
-    </gazebo>
-    <joint name="caster_${sub}_joint" type="fixed">
-      <parent link="${parent}"/>
-      <child link="caster_${sub}"/>
-      <origin xyz="${transX} ${transY} ${transZ}" rpy="0 0 0" />
+  <joint name="caster_support_joint" type="continuous">
+    <axis xyz="0 0 1"/>
+    <parent link="base_link"/>
+    <child link="caster_support"/>
+    <origin xyz="0.15  0.0 -0.075" rpy="0 0 0"/>
+  </joint>
+  <link name="caster_support">
+    <visual name="visual">
+      <geometry>
+        <box size="0.01 0.01 0.01"/>
+      </geometry>
+    </visual>
+    </link>
+  <joint type="continuous" name="caster_joint">
+    <!-- <origin xyz="0 -0.15 0.075" rpy="0 0 0"/> -->
+    <!-- <origin xyz="0 0.0 -0.10" rpy="0 1.5707 1.5707"/> -->
+    <!-- <origin xyz="0 -0.15 -0.05" rpy="1.57 0 0"/> -->
+    <origin xyz="0.0 0.0 0.0" rpy="1.57 0 0"/>
+    <child link="caster"></child>
+    <parent link="caster_support"></parent>
+    <axis xyz="0 0 1"/>
+    <limit effort="100" velocity="100.0"  lower="-5000" upper="5000" />
+  </joint>
+  <link name="left_wheel">
+    <collision name="collision">
+      <!-- <origin xyz="0 0.0 -0.10" rpy="0 1.5707 1.5707"/> -->
+      <geometry>
+         <cylinder  length="0.03" radius="0.0725"/>
+      </geometry>
+    </collision>
+    <visual name="visual">
+      <!-- <origin xyz="0 0.0 -0.10" rpy="0 0 0"/> -->
+      <geometry>
+        <cylinder  length="0.03" radius="0.0725"/>
+      </geometry>
+    </visual>
+    <inertial>
+      <mass value="1" />
+      <origin xyz="0.15 0.15 -0.05" rpy="1.57 0.0 0.0"/>
+      <inertia ixx="0.1" ixy="0" ixz="0" iyy="0.1" iyz="0" izz="0.1" />
+    </inertial>
+  </link>
+  <joint type="continuous" name="left_wheel_joint">
+    <!-- <origin xyz="0 0.15 0.075" rpy="0 0 0"/> -->
+    <origin xyz="-0.15 0.15 -0.05" rpy="1.57 0 0"/>
+    <child link="left_wheel"></child>
+    <parent link="base_link"></parent>
+    <axis xyz="0 0 1"/>
+    <limit effort="100" velocity="100.0"  lower="-5000" upper="5000" />
+  </joint>
+  <!--link name="visual_right_wheel">
+    <visual name="visual">
+      <origin xyz="0 0.0 0" rpy="0 1.5707 1.5707"/>
+      <geometry>
+        <cylinder  length="0.03" radius="0.0725"/>
+      </geometry>
+    </visual>
+  </link>
+  <joint type="fixed" name="visual_right_wheel_joint">
+    <origin xyz="0.15 -0.15 0.075" rpy="0 0 0"/>
+    <child link="visual_right_wheel">visual_right_wheel</child>
+    <parent link="base_link">base_link</parent>
+    <axis xyz="0 1 0"/>
+  </joint-->
+  <link name="right_wheel">
+    <collision name="collision">
+      <!-- <origin xyz="0 0.0 -0.10" rpy="0 1.5707 1.5707"/> -->
+      <!-- <origin xyz="0 0.15 -0.05" rpy="1.57 0 0"/> -->
+      <geometry>
+         <cylinder  length="0.03" radius="0.0725"/>
+      </geometry>
+    </collision>
+    <visual name="visual">
+      <!-- <origin xyz="0 0.0 -0.10" rpy="0 1.5707 1.5707"/> -->
+      <geometry>
+        <cylinder  length="0.03" radius="0.0725"/>
+      </geometry>
+    </visual>
+    <inertial>
+      <mass value="1" />
+      <origin xyz="0 0.0 0"/>
+      <inertia ixx="0.1" ixy="0" ixz="0" iyy="0.1" iyz="0" izz="0.1" />
+    </inertial>
+  </link>
+  <joint type="continuous" name="right_wheel_joint">
+    <!-- <origin xyz="0 -0.15 0.075" rpy="0 0 0"/> -->
+    <!-- <origin xyz="0 0.0 -0.10" rpy="0 1.5707 1.5707"/> -->
+    <origin xyz="-0.15 -0.15 -0.05" rpy="1.57 0 0"/>
+    <child link="right_wheel"></child>
+    <parent link="base_link"></parent>
+    <axis xyz="0 0 1"/>
+    <limit effort="100" velocity="100.0"  lower="-5000" upper="5000" />
+  </joint>
+  <xacro:sensor_hokuyo name="hokuyo" parent="base_link" size="0.05 0.05 0.05">
+    <origin xyz="0.25 0 0.1" rpy="0 0 0"/>
+  </xacro:sensor_hokuyo>
+  <transmission name="tran1">
+    <type>transmission_interface/SimpleTransmission</type>
+    <joint name="left_wheel_joint">
+      <hardwareInterface>VelocityJointInterface</hardwareInterface>
     </joint>
-  </xacro:macro>
+    <actuator name="left_motor">
+      <hardwareInterface>VelocityJointInterface</hardwareInterface>
+      <mechanicalReduction>1</mechanicalReduction>
+    </actuator>
+  </transmission>
+  <transmission name="tran2">
+    <type>transmission_interface/SimpleTransmission</type>
+    <joint name="right_wheel_joint">
+      <hardwareInterface>VelocityJointInterface</hardwareInterface>
+    </joint>
+    <actuator name="right_motor">
+      <hardwareInterface>VelocityJointInterface</hardwareInterface>
+      <mechanicalReduction>1</mechanicalReduction>
+    </actuator>
+  </transmission>
 </robot>
