Commit message: Simulate the gamma camera as a wide-angle fisheye
orne_gamma.gazebo: camera -> wideanglecamera with an equidistant lens
(hfov 2.3 -> 2.62, cutoff 2.1), drop the radial distortion block and
plugin K coefficients, near clip 0.03 -> 0.001, update rate 30 -> 20 Hz.
Lower the camera mount 0.565 -> 0.365 m in orne_gamma.urdf.xacro.

Co-Authored-By: Claude Sonnet 5 <noreply@anthropic.com>

File: orne_description/urdf/gamma/orne_gamma.urdf.xacro (robot description, xacro)
@@ -203,5 +203,5 @@
   </transmission>
   <joint name="camera_joint" type="fixed">
-    <origin xyz="0.223 -0.011 0.565" rpy="0 0.124 0"/>
+    <origin xyz="0.223 -0.011 0.365" rpy="0 0.124 0"/>
     <parent link="base_link"/>
     <child link="camera_link"/>
