Commit message: Fix caster material name and trailing newline
Reference the lowercase "black" material that is actually defined, and
add the missing end-of-file newline.

Co-Authored-By: Claude Sonnet 5 <noreply@anthropic.com>

File: orne_description/urdf/gamma/orne_gamma_caster.urdf.xacro (robot description, xacro)
@@ -14,5 +14,5 @@
           <sphere radius="${caster_radius}" />
         </geometry>
-        <material name="Black" />
+        <material name="black" />
       </visual>
       <collision>
